File: projects/basic-emulator/schematic/basic-emulator.kicad_pcb (KiCad board)
At the start: 2 copper layers, 44.2 x 61.7 mm, 21 parts

Commit message: Restructure Repository
Parts:
- added G***: LOGO, CustomSymbols:Github-QR-Code, B.Cu at (155.8, 100.0)
- added G***: LOGO, CustomSymbols:OSSHW-Symbol, B.Cu at (190.2, 100.8)
- added R2: 500, Resistor_SMD:R_1206_3216Metric_Pad1.30x1.75mm_HandSolder, F.Cu at (151.2, 68.2)
- added SW1: SW_SPST, Button_Switch_THT:SW_DIP_SPSTx01_Slide_9.78x4.72mm_W7.62mm_P2.54mm, F.Cu at (159.1, 62.8)
Connections:
- A1 pad 1: Net-(A1-GPIO0) -> unconnected-(A1-GPIO0-Pad1)
- A1 pad 2: unconnected-(A1-GPIO1-Pad2) -> Net-(A1-GPIO1)
- A1 pad 36: unconnected-(A1-3V3-Pad36) -> +3V3
- A1 pad 6: unconnected-(A1-GPIO4-Pad6) -> Net-(A1-GPIO4)
- R1 pad 2: Net-(A1-GPIO0) -> Net-(A1-GPIO4)
Routing:
- net +3V3: track 0.00 -> 27.9 mm
- net GND: track 188.1 -> 213.1 mm
- net Net-(A1-GPIO1): track 0.00 -> 20.8 mm
- net Net-(A1-GPIO0): track 16.1 -> 0.00 mm
- net Net-(A1-GPIO4): track 0.00 -> 4.24 mm
- net unconnected-(A1-GPIO1-Pad2): track 0.80 -> 0.00 mm
- net unconnected-(A1-GPIO0-Pad1): track 0.00 -> 0.80 mm
- net unconnected-(A1-3V3-Pad36): track 0.80 -> 0.00 mm
- removed copper zone on B.Cu, net GND
Other:
- board size 44.2 x 61.7 mm -> 47 x 61.7 mm
- rule pad_to_mask_clearance: 0 -> 0.0508
- board text added: "ON"
- board text added: "ON: Xbox OFF: PS3/Wii U"
