File: projects/basic-emulator/schematic/basic-emulator.kicad_sch (KiCad schematic)
At the start: 19 parts, among them SW1 SW_SPST

Commit message: Restructure Repository
Parts:
- SW1: footprint (none) -> Button_Switch_THT:SW_DIP_SPSTx01_Slide_9.78x4.72mm_W7.62mm_P2.54mm
Connections:
- net at A1.1 (GPIO0): no longer R1.2
- net at A1.2 (GPIO1): now also R2.1, SW1.2 (B)
- net at A1.6 (GPIO4): now also R1.2
- now unconnected: A1.21 (GPIO16)
Other:
- moved on the sheet: R2, SW1
Changed lines of the file:
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@@
-	)
-	(junction
-		(at 345.44 180.34)
-		(diameter 0)
-		(color 0 0 0 0)
 	)
 	(junction
@@
 	)
 	(junction
+		(at 261.62 180.34)
+		(diameter 0)
+		(color 0 0 0 0)
+	)
+	(junction
 		(at 215.9 134.62)
 		(diameter 0)
@@
 	(wire
 		(pts
+			(xy 261.62 180.34) (xy 275.59 180.34)
+		)
+		(stroke
+			(width 0)
+			(type default)
+		)
+	)
+	(wire
+		(pts
 			(xy 215.9 107.95) (xy 215.9 113.03)
 		)
@@
 	(wire
 		(pts
-			(xy 240.03 313.69) (xy 266.7 313.69)
+			(xy 240.03 313.69) (xy 267.97 313.69)
 		)
 		(stroke
@@
 	(wire
 		(pts
-			(xy 275.59 177.8) (xy 266.7 177.8)
-		)
-		(stroke
-			(width 0)
-			(type default)
-		)
-	)
-	(wire
-		(pts
 			(xy 210.82 266.7) (xy 210.82 285.75)
 		)
@@
 	(wire
 		(pts
-			(xy 356.87 180.34) (xy 361.95 180.34)
+			(xy 267.97 187.96) (xy 267.97 313.69)
+		)
+		(stroke
+			(width 0)
+			(type default)
+		)
+	)
+	(wire
+		(pts
+			(xy 250.19 180.34) (xy 247.65 180.34)
 		)
 		(stroke
@@
 	(wire
 		(pts
-			(xy 361.95 180.34) (xy 361.95 176.53)
+			(xy 247.65 180.34) (xy 247.65 176.53)
 		)
 		(stroke
@@
 	(wire
 		(pts
+			(xy 275.59 187.96) (xy 267.97 187.96)
+		)
+		(stroke
+			(width 0)
+			(type default)
+		)
+	)
+	(wire
+		(pts
 			(xy 303.53 149.86) (xy 303.53 154.94)
 		)
@@
 	(wire
 		(pts
-			(xy 345.44 180.34) (xy 346.71 180.34)
+			(xy 261.62 180.34) (xy 260.35 180.34)
 		)
 		(stroke
@@
 	(wire
 		(pts
-			(xy 345.44 180.34) (xy 345.44 184.15)
-		)
-		(stroke
-			(width 0)
-			(type default)
-		)
-	)
-	(wire
-		(pts
-			(xy 321.31 180.34) (xy 345.44 180.34)
+			(xy 261.62 180.34) (xy 261.62 184.15)
 		)
 		(stroke
@@
 	(wire
 		(pts
-			(xy 266.7 177.8) (xy 266.7 313.69)
-		)
-		(stroke
-			(width 0)
-			(type default)
-		)
-	)
-	(wire
-		(pts
 			(xy 210.82 266.7) (xy 215.9 266.7)
 		)
@@
 	(wire
 		(pts
-			(xy 345.44 191.77) (xy 345.44 195.58)
+			(xy 261.62 191.77) (xy 261.62 195.58)
 		)
 		(stroke
@@
 	(symbol
 		(lib_id "Switch:SW_SPST")
-		(at 351.79 180.34 180)
+		(at 255.27 180.34 0)
+		(mirror x)
 		(unit 1)
 		(exclude_from_sim no)
@@
 		(fields_autoplaced yes)
 		(property "Reference" "SW1"
-			(at 351.79 175.26 0)
+			(at 255.27 175.26 0)
 			(effects
 				(font
@@
 		)
 		(property "Value" "SW_SPST"
-			(at 351.79 177.8 0)
-			(effects
-				(font
-					(size 1.27 1.27)
-				)
-			)
-		)
-		(property "Footprint" ""
-			(at 351.79 180.34 0)
+			(at 255.27 177.8 0)
+			(effects
+				(font
+					(size 1.27 1.27)
+				)
+			)
+		)
+		(property "Footprint" "Button_Switch_THT:SW_DIP_SPSTx01_Slide_9.78x4.72mm_W7.62mm_P2.54mm"
+			(at 255.27 180.34 0)
 			(effects
 				(font
@@
 		)
 		(property "Datasheet" "~"
-			(at 351.79 180.34 0)
+			(at 255.27 180.34 0)
 			(effects
 				(font
@@
 		)
 		(property "Description" "Single Pole Single Throw (SPST) switch"
-			(at 351.79 180.34 0)
+			(at 255.27 180.34 0)
 			(effects
 				(font
@@
 	(symbol
 		(lib_id "power:+3V3")
-		(at 361.95 176.53 0)
+		(at 247.65 176.53 0)
+		(mirror y)
 		(unit 1)
 		(exclude_from_sim no)
@@
 		(fields_autoplaced yes)
 		(property "Reference" "#PWR014"
-			(at 361.95 180.34 0)
+			(at 247.65 180.34 0)
 			(effects
 				(font
@@
 		)
 		(property "Value" "+3V3"
-			(at 361.95 171.45 0)
+			(at 247.65 171.45 0)
 			(effects
 				(font
@@
 		)
 		(property "Footprint" ""
-			(at 361.95 176.53 0)
+			(at 247.65 176.53 0)
 			(effects
 				(font
@@
 		)
 		(property "Datasheet" ""
-			(at 361.95 176.53 0)
+			(at 247.65 176.53 0)
 			(effects
 				(font
@@
 		)
 		(property "Description" "Power symbol creates a global label with name \"+3V3\""
-			(at 361.95 176.53 0)
+			(at 247.65 176.53 0)
 			(effects
 				(font
@@
 	(symbol
 		(lib_id "Device:R_US")
-		(at 345.44 187.96 0)
+		(at 261.62 187.96 0)
+		(mirror y)
 		(unit 1)
 		(exclude_from_sim no)
@@
 		(fields_autoplaced yes)
 		(property "Reference" "R2"
-			(at 347.98 186.6899 0)
+			(at 259.08 186.6899 0)
 			(effects
 				(font
@@
 		)
 		(property "Value" "500"
-			(at 347.98 189.2299 0)
+			(at 259.08 189.2299 0)
 			(effects
 				(font
@@
 		)
 		(property "Footprint" "Resistor_SMD:R_1206_3216Metric_Pad1.30x1.75mm_HandSolder"
-			(at 346.456 188.214 90)
+			(at 260.604 188.214 90)
 			(effects
 				(font
@@
 		)
 		(property "Datasheet" "~"
-			(at 345.44 187.96 0)
+			(at 261.62 187.96 0)
 			(effects
 				(font
@@
 		)
 		(property "Description" "Resistor, US symbol"
-			(at 345.44 187.96 0)
+			(at 261.62 187.96 0)
 			(effects
 				(font
@@
 	(symbol
 		(lib_id "power:GND")
-		(at 345.44 195.58 0)
+		(at 261.62 195.58 0)
+		(mirror y)
 		(unit 1)
 		(exclude_from_sim no)
@@
 		(fields_autoplaced yes)
 		(property "Reference" "#PWR015"
-			(at 345.44 201.93 0)
+			(at 261.62 201.93 0)
 			(effects
 				(font
@@
 		)
 		(property "Value" "GND"
-			(at 345.44 200.66 0)
+			(at 261.62 200.66 0)
 			(effects
 				(font
@@
 		)
 		(property "Footprint" ""
-			(at 345.44 195.58 0)
+			(at 261.62 195.58 0)
 			(effects
 				(font
@@
 		)
 		(property "Datasheet" ""
-			(at 345.44 195.58 0)
+			(at 261.62 195.58 0)
 			(effects
 				(font
@@
 		)
 		(property "Description" "Power symbol creates a global label with name \"GND\" , ground"
-			(at 345.44 195.58 0)
-			(effects
-				(font
+			(at 261.62 195.58 0)
+			(effects
+				(font
